Commit message: attempting to begin lidar

File: olin_description/urdf/camera.urdf.xacro (robot description, xacro)
@@ -26,5 +26,5 @@
 		<joint name="$camera_${camera_id}_joint" type="fixed">
 			<axis xyz="0 1 0" />
-			<origin xyz="0.05 0 0.4" rpy="0 0 -1.57"/>
+			<origin xyz="0 -0.3 0.2" rpy="0 0 -1.57"/>
 			<parent link="base_link"/>
 			<child link="camera_${camera_id}_link"/>

File: olin_description/urdf/robot.urdf.xacro (robot description, xacro)
@@ -3,4 +3,5 @@
 	<xacro:include filename="$(find olin_description)/urdf/wheel.urdf.xacro" />
 	<xacro:include filename="$(find olin_description)/urdf/camera.urdf.xacro" />
+	<xacro:include filename="$(find olin_description)/urdf/lidar.urdf.xacro" />
 	<property name="M_PI" value="3.14159"/>
 	<gazebo>
@@ -45,3 +46,5 @@
 	<!-- Camera -->
 	<xacro:simple_camera camera_id="1"/>
+	<!-- LIDAR -->
+	<xacro:lidar lidar_id="1"/>
 </robot>

Commit message: fixed robot configuration (better fit differential drive); better rotation; equation-driven-urdf

File: olin_description/urdf/camera.urdf.xacro (robot description, xacro)
@@ -26,5 +26,5 @@
 		<joint name="$camera_${camera_id}_joint" type="fixed">
 			<axis xyz="0 1 0" />
-			<origin xyz="0 -0.3 0.2" rpy="0 0 -1.57"/>
+			<origin xyz="${base_xdim} 0 0.2" rpy="0 0 0"/> <!-- NOT SO SURE -->
 			<parent link="base_link"/>
 			<child link="camera_${camera_id}_link"/>
@@ -34,5 +34,5 @@
 				<update_rate>30.0</update_rate>
 				<camera>
-					<horizontal_fov>1.3962634</horizontal_fov>
+					<horizontal_fov>1.186</horizontal_fov>
 					<image>
 						<width>800</width>

File: olin_description/urdf/lidar.urdf.xacro (robot description, xacro)
@@ -3,6 +3,6 @@
 	<xacro:macro name="lidar" params="lidar_id">
 		<joint name="hokuyo_joint" type="fixed">
-			<axis xyz="0 1 0" />
-			<origin xyz="0 -0.3 0.2" rpy="0 0 -1.57"/>
+			<axis xyz="0 1 0" /> <!-- NOT SO SURE -->
+			<origin xyz="${base_xdim} 0 0.2" rpy="0 0 0"/>
 			<parent link="base_link"/>
 			<child link="hokuyo_link"/>

File: olin_description/urdf/robot.urdf.xacro (robot description, xacro)
@@ -5,4 +5,19 @@
 	<xacro:include filename="$(find olin_description)/urdf/lidar.urdf.xacro" />
 	<property name="M_PI" value="3.14159"/>
+	<property name="wheel_radius" value="0.1"/>
+	<property name="wheel_thickness" value="0.04"/>
+	<property name="wheel_x_offset" value="0.11"/>
+	<property name="wheel_y_offset" value="0.19"/>
+	<property name="wheel_mass" value="0.1"/>
+	<property name="base_xdim" value="0.4"/>
+	<property name="base_ydim" value="0.3"/>
+	<property name="base_zdim" value="0.1"/>
+	<property name="base_mass" value="2"/>
+	<xacro:macro name="box_inertia" params="m x y z">
+		<inertia  ixx="${m*(y*y+z*z)/12}" ixy = "0" ixz = "0"
+			iyy="${m*(x*x+z*z)/12}" iyz = "0"
+			izz="${m*(x*x+z*z)/12}"
+			/>
+	</xacro:macro>
 	<gazebo>
 		<plugin name="gazebo_ros_control" filename="libgazebo_ros_control.so">
@@ -15,5 +30,5 @@
 		<visual>
 			<geometry>
-				<box size="0.3 0.6 0.1"/>
+				<box size="${base_xdim} ${base_ydim} ${base_zdim}"/>
 			</geometry>
 			<material name="white">
@@ -23,24 +38,24 @@
 		<collision>
 			<geometry>
-				<box size="0.3 0.6 0.1"/>
+				<box size="${base_xdim} ${base_ydim} ${base_zdim}"/>
 			</geometry>
 		</collision>
 		<inertial>
-			<mass value="1.8"/>
-			<inertia ixx="0.015" ixy="0" ixz="0" iyy="0.015" iyz="0" izz="0.0675"/>
+			<mass value="${base_mass}"/>
+			<box_inertia m="${base_mass}" x="${base_xdim}" y="${base_ydim}" z="${base_zdim}"/>
 		</inertial>
 	</link>
 	<!-- Four Wheels -->
 	<xacro:wheel wheel_prefix="front_left">
-		<origin xyz="0.19 0.3 0" rpy="0 0 0"/>
+		<origin xyz="${wheel_x_offset} ${wheel_y_offset} 0" rpy="0 0 0"/>
 	</xacro:wheel>
 	<xacro:wheel wheel_prefix="front_right">
-		<origin xyz="-0.19 0.3 0" rpy="0 0 0"/>
+		<origin xyz="${wheel_x_offset} -${wheel_y_offset} 0" rpy="0 0 0"/>
 	</xacro:wheel>
 	<xacro:wheel wheel_prefix="back_left">
-		<origin xyz="0.19 -0.3 0" rpy="0 0 0"/>
+		<origin xyz="-${wheel_x_offset} ${wheel_y_offset} 0" rpy="0 0 0"/>
 	</xacro:wheel>
 	<xacro:wheel wheel_prefix="back_right">
-		<origin xyz="-0.19 -0.3 0" rpy="0 0 0"/>
+		<origin xyz="-${wheel_x_offset} -${wheel_y_offset} 0" rpy="0 0 0"/>
 	</xacro:wheel>
 	<!-- Camera -->

File: olin_description/urdf/wheel.urdf.xacro (robot description, xacro)
@@ -1,14 +1,20 @@
 <?xml version="1.0"?>
 <robot xmlns:xacro="http://ros.org/wifi/xacro" name="wheel">
+	<xacro:macro name="cylinder_inertia" params="m r h">
+		<inertia  ixx="${m*(3*r*r+h*h)/12}" ixy = "0" ixz = "0"
+			iyy="${m*(3*r*r+h*h)/12}" iyz = "0"
+			izz="${m*r*r/2}"
+			/>
+	</xacro:macro>
 	<xacro:macro name="wheel" params="wheel_prefix *joint_pose">
 		<link name="${wheel_prefix}_wheel_link">
 			<inertial>
-				<mass value="0.0015"/>
-				<inertia ixx="3.64e-06" ixy="0" ixz="0" iyy="3.64e-06" iyz="0" izz="6.91e-06"/>
+				<mass value="${wheel_mass}"/>
+				<cylinder_inertia m="${wheel_mass}" r="${wheel_radius}" h="${wheel_thickness}"/>
 			</inertial>
 			<visual>
-				<origin xyz="0 0 0" rpy="0 ${M_PI/2} 0"/>
+				<origin xyz="0 0 0" rpy="${M_PI/2} 0 0"/>
 				<geometry>
-					<cylinder length="0.04" radius="0.1"/>
+					<cylinder length="${wheel_thickness}" radius="${wheel_radius}"/>
 				</geometry>
 				<material name="black">
@@ -17,7 +23,7 @@
 			</visual>
 			<collision>
-				<origin xyz="0.0 0.0 0" rpy="0 ${M_PI/2} 0"/>
+				<origin xyz="0.0 0.0 0" rpy="${M_PI/2} 0 0"/>
 				<geometry>
-					<cylinder length="0.04" radius="0.1"/>
+					<cylinder length="${wheel_thickness}" radius="${wheel_radius}"/>
 				</geometry>
 			</collision>
@@ -26,5 +32,5 @@
 			<mu1 value="1.0"/>
 			<mu2 value="1.0"/>
-			<kp value="10000000.0" />
+			<kp value="1000000.0" />
 			<kd value="1.0" />
 			<!--<fdir1 value="1 0 0"/>-->
@@ -36,5 +42,5 @@
 			<!--<origin xyz="0 0 0" rpy="0 0 0"/>-->
 			<!---<joint_properties damping="0.0" friction="0.5"/>-->
-			<axis xyz="1 0 0" rpy="0 0 0"/>
+			<axis xyz="0 1 0" rpy="0 0 0"/>
 		</joint>
 		<transmission name="${wheel_prefix}_wheel_trans">
