Commit message: added hokuyo mesh and fixed package dependencies (still needs to be fixed)

File: olin_description/urdf/lidar.urdf.xacro (robot description, xacro)
@@ -19,5 +19,5 @@
 				<origin xyz="0 0 0" rpy="0 0 0"/>
 				<geometry>
-					<mesh filename="package://rrbot_description/meshes/hokuyo.dae"/>
+					<mesh filename="package://olin_description/meshes/hokuyo.dae"/>
 				</geometry>
 			</visual>
