Commit message: added camera and fixed orientation for differential drive

File: olin_description/urdf/robot.urdf.xacro (robot description, xacro)
@@ -2,4 +2,5 @@
 <robot name="olin" xmlns:xacro="http://ros.org/wiki/xacro">
 	<xacro:include filename="$(find olin_description)/urdf/wheel.urdf.xacro" />
+	<xacro:include filename="$(find olin_description)/urdf/camera.urdf.xacro" />
 	<property name="M_PI" value="3.14159"/>
 	<gazebo>
@@ -9,4 +10,5 @@
 		</plugin>
 	</gazebo>
+	<!-- Root Element -->
 	<link name="base_link">
 		<visual>
@@ -28,15 +30,18 @@
 		</inertial>
 	</link>
+	<!-- Four Wheels -->
 	<xacro:wheel wheel_prefix="front_left">
+		<origin xyz="0.19 0.3 0" rpy="0 0 0"/>
+	</xacro:wheel>
+	<xacro:wheel wheel_prefix="front_right">
 		<origin xyz="-0.19 0.3 0" rpy="0 0 0"/>
 	</xacro:wheel>
-	<xacro:wheel wheel_prefix="front_right">
-		<origin xyz="0.19 0.3 0" rpy="0 0 0"/>
+	<xacro:wheel wheel_prefix="back_left">
+		<origin xyz="0.19 -0.3 0" rpy="0 0 0"/>
 	</xacro:wheel>
-	<xacro:wheel wheel_prefix="back_left">
+	<xacro:wheel wheel_prefix="back_right">
 		<origin xyz="-0.19 -0.3 0" rpy="0 0 0"/>
 	</xacro:wheel>
-	<xacro:wheel wheel_prefix="back_right">
-		<origin xyz="0.19 -0.3 0" rpy="0 0 0"/>
-	</xacro:wheel>
+	<!-- Camera -->
+	<xacro:simple_camera camera_id="1"/>
 </robot>

Commit message: added sonar

File: olin_description/urdf/robot.urdf.xacro (robot description, xacro)
@@ -5,4 +5,5 @@
 	<xacro:include filename="$(find olin_description)/urdf/lidar.urdf.xacro" />
 	<xacro:include filename="$(find olin_description)/urdf/imu.urdf.xacro" />
+	<xacro:include filename="$(find olin_description)/urdf/sonar.urdf.xacro" />
 	<property name="M_PI" value="3.14159"/>
 	<property name="wheel_radius" value="0.1"/>
@@ -66,3 +67,11 @@
 	<!-- IMU -->
 	<xacro:fake_imu />
+	<!-- Left Sonar -->
+	<xacro:sonar_sensor name="left_sonar" parent="base_link" ros_topic="left_sonar" update_rate="1" min_range="0.01" max_range="5.0" field_of_view="${M_PI/2}" ray_count="100" >
+		<origin xyz="0 ${base_ydim} 0" rpy="0 0 ${M_PI/2}" />
+	</xacro:sonar_sensor>
+	<!-- Right Sonar -->
+	<xacro:sonar_sensor name="right_sonar" parent="base_link" ros_topic="right_sonar" update_rate="1" min_range="0.01" max_range="5.0" field_of_view="${M_PI/2}" ray_count="100" >
+		<origin xyz="0 ${-base_ydim} 0" rpy="0 0 ${-M_PI/2}" />
+	</xacro:sonar_sensor>
 </robot>

File: olin_description/urdf/sonar.urdf.xacro (robot description, xacro)
@@ -16,49 +16,49 @@
         <origin xyz="0 0 0" rpy="0 0 0" />
         <geometry>
-          <!--<box size="0.01 0.01 0.01" /> -->
-          <mesh filename="package://hector_sensors_description/meshes/sonar_sensor/max_sonar_ez4.dae"/>
-        </geometry>
-      </visual>
-      <collision>
-        <origin xyz="0 0 0" rpy="0 0 0" />
-        <geometry>
-          <box size="0.01 0.01 0.01" />
-        </geometry>
-      </collision>
-    </link>
-    <gazebo reference="${name}_link">
-      <sensor type="ray" name="${name}">
-        <always_on>true</always_on>
-        <update_rate>${update_rate}</update_rate>
-        <pose>0 0 0 0 0 0</pose>
-        <visualize>false</visualize>
-        <ray>
-          <scan>
-            <horizontal>
-              <samples>${ray_count}</samples>
-              <resolution>1</resolution>
-              <min_angle>-${field_of_view/2}</min_angle>
-              <max_angle> ${field_of_view/2}</max_angle>
-            </horizontal>
-            <vertical>
-              <samples>${ray_count}</samples>
-              <resolution>1</resolution>
-              <min_angle>-${field_of_view/2}</min_angle>
-              <max_angle> ${field_of_view/2}</max_angle>
-            </vertical>
-          </scan>
-          <range>
-            <min>${min_range}</min>
-            <max>${max_range}</max>
-            <resolution>0.01</resolution>
-          </range>
-        </ray>
-        <plugin name="gazebo_ros_${name}_controller" filename="libhector_gazebo_ros_sonar.so">
-          <gaussianNoise>0.005</gaussianNoise>
-          <topicName>${ros_topic}</topicName>
-          <frameId>${name}_link</frameId>
-        </plugin>
-      </sensor>
-    </gazebo>
+			<!--<box size="0.01 0.01 0.01" /> -->
+			<mesh filename="package://hector_sensors_description/meshes/sonar_sensor/max_sonar_ez4.dae"/>
+		</geometry>
+	</visual>
+	<collision>
+		<origin xyz="0 0 0" rpy="0 0 0" />
+		<geometry>
+			<box size="0.01 0.01 0.01" />
+		</geometry>
+	</collision>
+</link>
+<gazebo reference="${name}_link">
+	<sensor type="ray" name="${name}">
+		<always_on>true</always_on>
+		<update_rate>${update_rate}</update_rate>
+		<pose>0 0 0 0 0 0</pose>
+		<visualize>false</visualize>
+		<ray>
+			<scan>
+				<horizontal>
+					<samples>${ray_count}</samples>
+					<resolution>1</resolution>
+					<min_angle>-${field_of_view/2}</min_angle>
+					<max_angle> ${field_of_view/2}</max_angle>
+				</horizontal>
+				<vertical>
+					<samples>${ray_count}</samples>
+					<resolution>1</resolution>
+					<min_angle>-${field_of_view/2}</min_angle>
+					<max_angle> ${field_of_view/2}</max_angle>
+				</vertical>
+			</scan>
+			<range>
+				<min>${min_range}</min>
+				<max>${max_range}</max>
+				<resolution>0.01</resolution>
+			</range>
+		</ray>
+		<plugin name="gazebo_ros_${name}_controller" filename="libhector_gazebo_ros_sonar.so">
+			<gaussianNoise>0.005</gaussianNoise>
+			<topicName>${ros_topic}</topicName>
+			<frameId>${name}_link</frameId>
+		</plugin>
+	</sensor>
+</gazebo>
   </xacro:macro>
 </robot>

Commit message: fixing Sonar, incorrect range readings

File: olin_description/urdf/robot.urdf.xacro (robot description, xacro)
@@ -5,15 +5,15 @@
 	<xacro:include filename="$(find olin_description)/urdf/lidar.urdf.xacro" />
 	<xacro:include filename="$(find olin_description)/urdf/imu.urdf.xacro" />
-	<xacro:include filename="$(find olin_description)/urdf/sonar.urdf.xacro" />
+	<xacro:include filename="$(find olin_description)/urdf/range.urdf.xacro" />
 	<property name="M_PI" value="3.14159"/>
-	<property name="wheel_radius" value="0.1"/>
+	<property name="wheel_radius" value="0.07"/>
 	<property name="wheel_thickness" value="0.04"/>
-	<property name="wheel_x_offset" value="0.11"/>
-	<property name="wheel_y_offset" value="0.19"/>
+	<property name="wheel_x_offset" value="0.25"/>
+	<property name="wheel_y_offset" value="0.29"/>
 	<property name="wheel_mass" value="0.1"/>
-	<property name="base_xdim" value="0.4"/>
-	<property name="base_ydim" value="0.3"/>
+	<property name="base_xdim" value="0.5"/>
+	<property name="base_ydim" value="0.5"/>
 	<property name="base_zdim" value="0.1"/>
-	<property name="base_mass" value="2"/>
+	<property name="base_mass" value="3"/>
 	<xacro:macro name="box_inertia" params="m x y z">
 		<inertia  ixx="${m*(y*y+z*z)/12}" ixy = "0" ixz = "0"
@@ -21,4 +21,17 @@
 			izz="${m*(x*x+z*z)/12}"
 			/>
+	</xacro:macro>
+	<xacro:macro name="sonar_sensor" params="name parent ros_topic *origin *pose">
+		<xacro:range_sensor name="${name}" parent="${parent}" ros_topic="${ros_topic}" update_rate="1" min_range="1.0" max_range="5.0" field_of_view="${M_PI/4}" ray_count="5">
+			<xacro:insert_block name="origin"/>
+			<xacro:insert_block name="pose"/>
+			<mesh filename="package://hector_sensors_description/meshes/sonar_sensor/max_sonar_ez4.dae"/>
+		</xacro:range_sensor>
+	</xacro:macro>
+	<xacro:macro name="ir_sensor" params="name parent ros_topic *origin">
+		<xacro:range_sensor name="${name}" parent="${parent}" ros_topic="${ros_topic}" update_rate="1" min_range="0.01" max_range="5.0" field_of_view="${M_PI/8}" ray_count="10">
+			<xacro:insert_block name="origin"/>
+			<mesh filename="package://hector_sensors_description/meshes/sonar_sensor/max_sonar_ez4.dae"/>
+		</xacro:range_sensor>
 	</xacro:macro>
 	<gazebo>
@@ -68,10 +81,11 @@
 	<xacro:fake_imu />
 	<!-- Left Sonar -->
-	<xacro:sonar_sensor name="left_sonar" parent="base_link" ros_topic="left_sonar" update_rate="1" min_range="0.01" max_range="5.0" field_of_view="${M_PI/2}" ray_count="100" >
-		<origin xyz="0 ${base_ydim} 0" rpy="0 0 ${M_PI/2}" />
+	<xacro:sonar_sensor name="left_sonar" parent="base_link" ros_topic="left_sonar">
+		<origin xyz="0 ${base_ydim/2} 0" rpy="0 ${M_PI/2} 0" />
+		<pose xyz="0 ${base_ydim/2} 0" rpy="0 ${M_PI/2} 0" />
 	</xacro:sonar_sensor>
 	<!-- Right Sonar -->
-	<xacro:sonar_sensor name="right_sonar" parent="base_link" ros_topic="right_sonar" update_rate="1" min_range="0.01" max_range="5.0" field_of_view="${M_PI/2}" ray_count="100" >
-		<origin xyz="0 ${-base_ydim} 0" rpy="0 0 ${-M_PI/2}" />
-	</xacro:sonar_sensor>
+	<!--<xacro:sonar_sensor name="right_sonar" parent="base_link" ros_topic="right_sonar">
+		<origin xyz="0 ${-base_ydim/2 - 0.02} 0" rpy="0 0 ${-M_PI/2}" />
+	</xacro:sonar_sensor>-->
 </robot>
