Commit message: fixed sonar ... by which I mean I figured out why it was giving the values it gave. It picked up collision signal with the ground! Since the robot is so low, well...

File: funrobo_description/urdf/range.urdf.xacro (robot description, xacro)
@@ -1,5 +1,5 @@
 <?xml version="1.0"?>
 <robot xmlns:xacro="http://ros.org/wiki/xacro">
-	<xacro:macro name="range_sensor" params="name parent *origin *pose *mesh ros_topic update_rate min_range max_range field_of_view ray_count">
+	<xacro:macro name="range_sensor" params="name parent *origin *mesh ros_topic update_rate min_range max_range field_of_view ray_count">
 		<joint name="${name}_joint" type="fixed">
 			<xacro:insert_block name="origin" />
@@ -8,5 +8,4 @@
 		</joint>
 		<link name="${name}_link">
-			<xacro:insert_block name="pose" />
 			<inertial>
 				<mass value="0.001" />
@@ -33,6 +32,6 @@
 				<always_on>true</always_on>
 				<update_rate>${update_rate}</update_rate>
-				<pose>0 0 0 0 0 1.57</pose>
-				<visualize>true</visualize>
+				<pose>0 0 0 0 0 0</pose>
+				<visualize>false</visualize>
 				<ray>
 					<scan>
@@ -57,5 +56,5 @@
 				</ray>
 				<plugin name="gazebo_ros_${name}_controller" filename="libhector_gazebo_ros_sonar.so">
-					<gaussianNoise>0.005</gaussianNoise>
+					<!--<gaussianNoise>0.005</gaussianNoise>-->
 					<topicName>${ros_topic}</topicName>
 					<frameId>${name}_link</frameId>

File: funrobo_description/urdf/robot.urdf.xacro (robot description, xacro)
@@ -22,8 +22,7 @@
 			/>
 	</xacro:macro>
-	<xacro:macro name="sonar_sensor" params="name parent ros_topic *origin *pose">
-		<xacro:range_sensor name="${name}" parent="${parent}" ros_topic="${ros_topic}" update_rate="1" min_range="1.0" max_range="5.0" field_of_view="${M_PI/4}" ray_count="5">
+	<xacro:macro name="sonar_sensor" params="name parent ros_topic *origin">
+		<xacro:range_sensor name="${name}" parent="${parent}" ros_topic="${ros_topic}" update_rate="1" min_range="0.25" max_range="7.65" field_of_view="${30 * M_PI/180}" ray_count="50">
 			<xacro:insert_block name="origin"/>
-			<xacro:insert_block name="pose"/>
 			<mesh filename="package://hector_sensors_description/meshes/sonar_sensor/max_sonar_ez4.dae"/>
 		</xacro:range_sensor>
@@ -82,10 +81,9 @@
 	<!-- Left Sonar -->
 	<xacro:sonar_sensor name="left_sonar" parent="base_link" ros_topic="left_sonar">
-		<origin xyz="0 ${base_ydim/2} 0" rpy="0 ${M_PI/2} 0" />
-		<pose xyz="0 ${base_ydim/2} 0" rpy="0 ${M_PI/2} 0" />
+		<origin xyz="0 ${base_ydim/2 + 0.02} 0" rpy="0 0 ${M_PI/2}" />
 	</xacro:sonar_sensor>
 	<!-- Right Sonar -->
-	<!--<xacro:sonar_sensor name="right_sonar" parent="base_link" ros_topic="right_sonar">
+	<xacro:sonar_sensor name="right_sonar" parent="base_link" ros_topic="right_sonar">
 		<origin xyz="0 ${-base_ydim/2 - 0.02} 0" rpy="0 0 ${-M_PI/2}" />
-	</xacro:sonar_sensor>-->
+	</xacro:sonar_sensor>
 </robot>
