Commit message: renamed everything from olin --> funrobo

File: funrobo_description/urdf/camera.urdf.xacro (robot description, xacro)
@@ -53,5 +53,5 @@
 					<alwaysOn>true</alwaysOn>
 					<updateRate>0.0</updateRate>
-					<cameraName>/olin/camera_${camera_id}</cameraName>
+					<cameraName>/funrobo/camera_${camera_id}</cameraName>
 					<imageTopicName>image_raw</imageTopicName>
 					<cameraInfoTopicName>camera_info</cameraInfoTopicName>

File: funrobo_description/urdf/lidar.urdf.xacro (robot description, xacro)
@@ -19,5 +19,5 @@
 				<origin xyz="0 0 0" rpy="0 0 0"/>
 				<geometry>
-					<mesh filename="package://olin_description/meshes/hokuyo.dae"/>
+					<mesh filename="package://funrobo_description/meshes/hokuyo.dae"/>
 				</geometry>
 			</visual>
@@ -54,5 +54,5 @@
 				</ray>
 				<plugin name="gazebo_ros_head_hokuyo_controller" filename="libgazebo_ros_laser.so">
-					<topicName>/olin/laser/scan</topicName>
+					<topicName>/funrobo/laser/scan</topicName>
 					<frameName>hokuyo_link</frameName>
 				</plugin>

File: funrobo_description/urdf/robot.urdf.xacro (robot description, xacro)
@@ -1,9 +1,9 @@
 <?xml version="1.0"?>
-<robot name="olin" xmlns:xacro="http://ros.org/wiki/xacro">
-	<xacro:include filename="$(find olin_description)/urdf/wheel.urdf.xacro" />
-	<xacro:include filename="$(find olin_description)/urdf/camera.urdf.xacro" />
-	<xacro:include filename="$(find olin_description)/urdf/lidar.urdf.xacro" />
-	<xacro:include filename="$(find olin_description)/urdf/imu.urdf.xacro" />
-	<xacro:include filename="$(find olin_description)/urdf/range.urdf.xacro" />
+<robot name="funrobo" xmlns:xacro="http://ros.org/wiki/xacro">
+	<xacro:include filename="$(find funrobo_description)/urdf/wheel.urdf.xacro" />
+	<xacro:include filename="$(find funrobo_description)/urdf/camera.urdf.xacro" />
+	<xacro:include filename="$(find funrobo_description)/urdf/lidar.urdf.xacro" />
+	<xacro:include filename="$(find funrobo_description)/urdf/imu.urdf.xacro" />
+	<xacro:include filename="$(find funrobo_description)/urdf/range.urdf.xacro" />
 	<property name="M_PI" value="3.14159"/>
 	<property name="wheel_radius" value="0.07"/>

Commit message: fixed model geometry and updated readme

File: funrobo_description/urdf/camera.urdf.xacro (robot description, xacro)
@@ -1,5 +1,11 @@
 <?xml version="1.0"?>
 <robot xmlns:xacro="http://ros.org/wiki/xacro" name="simple_camera">
-	<xacro:macro name="simple_camera" params="camera_id">
+	<xacro:macro name="simple_camera" params="camera_id *origin">
+		<joint name="$camera_${camera_id}_joint" type="fixed">
+			<axis xyz="0 1 0" />
+			<xacro:insert_block name="origin"/>
+			<parent link="base_link"/>
+			<child link="camera_${camera_id}_link"/>
+		</joint>
 		<link name="camera_${camera_id}_link">
 			<collision>
@@ -24,10 +30,4 @@
 			</inertial>
 		</link>
-		<joint name="$camera_${camera_id}_joint" type="fixed">
-			<axis xyz="0 1 0" />
-			<origin xyz="${base_xdim} 0 0.2" rpy="0 0 0"/> <!-- NOT SO SURE -->
-			<parent link="base_link"/>
-			<child link="camera_${camera_id}_link"/>
-		</joint>
 		<gazebo reference="camera_${camera_id}_link">
 			<sensor type="camera" name="camera_${camera_id}">

File: funrobo_description/urdf/imu.urdf.xacro (robot description, xacro)
@@ -16,10 +16,10 @@
 			<visual>
 				<geometry>
-					<box size="0.1 0.1 0.1"/>
+					<box size="0.01 0.01 0.01"/>
 				</geometry>
 			</visual>
 			<collision>
 				<geometry>
-					<box size="0.1 0.1 0.1"/>
+					<box size="0.01 0.01 0.01"/>
 				</geometry>
 			</collision>

File: funrobo_description/urdf/lidar.urdf.xacro (robot description, xacro)
@@ -1,8 +1,8 @@
 <?xml version="1.0"?>
 <robot xmlns:xacro="http://ros.org/wiki/xacro" name="lidar">
-	<xacro:macro name="lidar" params="lidar_id">
+	<xacro:macro name="lidar" params="lidar_id *origin">
 		<joint name="hokuyo_joint" type="fixed">
 			<axis xyz="0 1 0" /> <!-- NOT SO SURE -->
-			<origin xyz="${base_xdim} 0 0.2" rpy="0 0 0"/>
+			<xacro:insert_block name="origin"/>
 			<parent link="base_link"/>
 			<child link="hokuyo_link"/>
@@ -36,13 +36,13 @@
 					<scan>
 						<horizontal>
-							<samples>720</samples>
+							<samples>1024</samples>
 							<resolution>1</resolution>
-							<min_angle>-1.570796</min_angle>
-							<max_angle>1.570796</max_angle>
+							<min_angle>-2.094395</min_angle>
+							<max_angle>2.094395</max_angle>
 						</horizontal>
 					</scan>
 					<range>
 						<min>0.1</min>
-						<max>10.0</max>
+						<max>6.0</max>
 						<resolution>0.1</resolution>
 					</range>

File: funrobo_description/urdf/robot.urdf.xacro (robot description, xacro)
@@ -30,5 +30,5 @@
 	</xacro:macro>
 	<xacro:macro name="ir_sensor" params="name parent ros_topic *origin">
-		<xacro:range_sensor name="${name}" parent="${parent}" ros_topic="${ros_topic}" update_rate="1" min_range="0.01" max_range="5.0" field_of_view="${M_PI/8}" ray_count="10">
+		<xacro:range_sensor name="${name}" parent="${parent}" ros_topic="${ros_topic}" update_rate="1" min_range="0.1" max_range="0.8" field_of_view="${8 * M_PI/180}" ray_count="10">
 			<xacro:insert_block name="origin"/>
 			<mesh filename="package://hector_sensors_description/meshes/sonar_sensor/max_sonar_ez4.dae"/>
@@ -75,7 +75,11 @@
 	</xacro:wheel>
 	<!-- Camera -->
-	<xacro:simple_camera camera_id="1"/>
+	<xacro:simple_camera camera_id="1">
+		<origin xyz="${base_xdim/2 - 0.1} 0 0.3" rpy="0 0 0"/>
+	</xacro:simple_camera>
 	<!-- LIDAR -->
-	<xacro:lidar lidar_id="1"/>
+	<xacro:lidar lidar_id="1">
+		<origin xyz="${base_xdim/2 - 0.02} 0 0.2" rpy="0 0 0"/>
+	</xacro:lidar>
 	<!-- IMU -->
 	<xacro:fake_imu />
@@ -88,3 +92,7 @@
 		<origin xyz="0 ${-base_ydim/2 - 0.02} 0" rpy="0 0 ${-M_PI/2}" />
 	</xacro:sonar_sensor>
+	<!-- Front-Down IR -->
+	<xacro:ir_sensor name="front_ir" parent="base_link" ros_topic="funrobo/front_ir">
+		<origin xyz="${base_xdim/2 + 0.02} 0 0" rpy="0 0 0" />
+	</xacro:ir_sensor>
 </robot>
